Commit message: feat: Add latest booster k1 robot model

File: src/holosoma/holosoma/data/robots/k1/k1_22dof-zed.urdf (robot description, URDF)
Before this commit: robot K1, 23 links, 22 joints
Links:
- link Head_2: mass 0.70 -> 0.781574; geometry collision mesh filename=meshes/Head_2_ZED.STL; visual mesh filename=meshes/Head_2_ZED.STL

File: src/holosoma/holosoma/data/robots/k1/k1_locomotion.urdf (robot description, URDF)
Before this commit: robot K1, 23 links, 22 joints
Joints:
- joint AAHead_yaw: type revolute -> fixed
- joint ALeft_Shoulder_Pitch: type revolute -> fixed
- joint ARight_Shoulder_Pitch: type revolute -> fixed
- joint Head_pitch: type revolute -> fixed
- joint Left_Elbow_Pitch: type revolute -> fixed
- joint Left_Elbow_Yaw: type revolute -> fixed
- joint Left_Shoulder_Roll: type revolute -> fixed
- joint Right_Elbow_Pitch: type revolute -> fixed
- joint Right_Elbow_Yaw: type revolute -> fixed
- joint Right_Shoulder_Roll: type revolute -> fixed
